File: tester.sch (EAGLE design)
At the start: 227 parts, among them Q2 16MHz, U1 VO1400AEFTR, U2 VO1400AEFTR, U3 VO1400AEFTR, U4 VO1400AEFTR, U5 VO1400AEFTR, U6 VO1400AEFTR, U7 VO1400AEFTR, U8 VO1400AEFTR

Commit message: Final tweaks before ordering
Parts:
- removed Q2: 16MHz, crystal:CRYTALHC49S
- R1, R10, R11, R12, R13, R14, R15, R16, R17, R18, R19, R2, R20, R21, R22, R23, R24, R25, R26, R3, R4, R5, R6, R7, R8, R9: value 1K -> 200
- R27, R28, R29, R30, R31, R32, R33, R34: value 1K -> 768
- R35, R36, R37, R38, R39, R40, R41, R42, R43, R44, R45, R46, R47, R48, R49, R50: value 1K -> 187
Connections:
- removed net N$6: Q2.1
- removed net N$7: Q2.2
Other:
- note added: "Green LED: 1318243 187 Ohm Red LED: 8529949 200 Ohm Orange LED: 8529922 200 Ohm Yellow LED: 1318247 200 Ohm"
